File: 001/001.kicad_pcb (KiCad board)
At the start: 2 copper layers, 101.6 x 53.3 mm, 13 parts, among them P1 Digital, P10 CONN_01X01, P11 CONN_01X01, P12 CONN_01X01, P13 CONN_01X01, P2 Power, P3 Analog, P4 Analog, P5 PWM, P6 PWM, P7 Communication, P8 CONN_01X01, P9 CONN_01X01

Commit message: 回路だいたい出来た。
Parts:
- added D1: 1N4148, Diode_THT:D_DO-35_SOD27_P7.62mm_Horizontal, F.Cu at (190.5, 133.3)
- added D2: 1N4148, Diode_THT:D_DO-35_SOD27_P7.62mm_Horizontal, F.Cu at (132.7, 156.8)
- added D3: 1N4148, Diode_THT:D_DO-35_SOD27_P7.62mm_Horizontal, F.Cu at (132.8, 186.0)
- added D4: D, Diode_THT:D_DO-35_SOD27_P10.16mm_Horizontal, F.Cu at (108.6, 170.4)
- added J1: LCD 2004, Connector_PinHeader_2.54mm:PinHeader_1x16_P2.54mm_Vertical, F.Cu at (104.7, 133.9)
- added J2: Relay OUT, Connector_JST:JST_XH_B9B-XH-A_1x09_P2.50mm_Vertical, F.Cu at (105.8, 177.7)
- added J3: iM920, Connector_JST:JST_XH_B7B-XH-A_1x07_P2.50mm_Vertical, F.Cu at (134.6, 134.9)
- added J4: GPS, Connector_JST:JST_XH_B5B-XH-A_1x05_P2.50mm_Vertical, F.Cu at (110.5, 164.2)
- added JA0: Conn_01x03, Connector_JST:JST_XH_B3B-XH-A_1x03_P2.50mm_Vertical, F.Cu at (161.0, 150.6)
- added JA1: Conn_01x03, Connector_JST:JST_XH_B3B-XH-A_1x03_P2.50mm_Vertical, F.Cu at (105.8, 193.3)
- added JA10: Conn_01x03, Connector_JST:JST_XH_B3B-XH-A_1x03_P2.50mm_Vertical, F.Cu at (117.8, 193.3)
- added JA11: Conn_01x03, Connector_JST:JST_XH_B3B-XH-A_1x03_P2.50mm_Vertical, F.Cu at (163.5, 142.8)
- added JA12: Conn_01x03, Connector_JST:JST_XH_B3B-XH-A_1x03_P2.50mm_Vertical, F.Cu at (132.8, 172.0)
- added JA13: Conn_01x03, Connector_JST:JST_XH_B3B-XH-A_1x03_P2.50mm_Vertical, F.Cu at (134.7, 179.8)
- added JA14: Conn_01x03, Connector_JST:JST_XH_B3B-XH-A_1x03_P2.50mm_Vertical, F.Cu at (149.1, 150.6)
- added JA15: Conn_01x03, Connector_JST:JST_XH_B3B-XH-A_1x03_P2.50mm_Vertical, F.Cu at (175.4, 142.8)
- added JA2: Conn_01x03, Connector_JST:JST_XH_B3B-XH-A_1x03_P2.50mm_Vertical, F.Cu at (129.7, 193.3)
- added JA3: Conn_01x03, Connector_JST:JST_XH_B3B-XH-A_1x03_P2.50mm_Vertical, F.Cu at (156.6, 134.9)
- added JA4: Conn_01x03, Connector_JST:JST_XH_B3B-XH-A_1x03_P2.50mm_Vertical, F.Cu at (159.2, 166.2)
- added JA5: Conn_01x03, Connector_JST:JST_XH_B3B-XH-A_1x03_P2.50mm_Vertical, F.Cu at (159.2, 158.3)
- added JA6: Conn_01x03, Connector_JST:JST_XH_B3B-XH-A_1x03_P2.50mm_Vertical, F.Cu at (180.4, 134.9)
- added JA7: Conn_01x03, Connector_JST:JST_XH_B3B-XH-A_1x03_P2.50mm_Vertical, F.Cu at (147.2, 158.3)
- added JA8: Conn_01x03, Connector_JST:JST_XH_B3B-XH-A_1x03_P2.50mm_Vertical, F.Cu at (168.5, 134.9)
- added JA9: Conn_01x03, Connector_JST:JST_XH_B3B-XH-A_1x03_P2.50mm_Vertical, F.Cu at (146.7, 173.9)
- added JC1: Conn_01x04, Connector_JST:JST_XH_B4B-XH-A_1x04_P2.50mm_Vertical, F.Cu at (105.8, 185.5)
- added JC2: Conn_01x04, Connector_JST:JST_XH_B4B-XH-A_1x04_P2.50mm_Vertical, F.Cu at (134.6, 150.6)
- added JC3: Conn_01x04, Connector_JST:JST_XH_B4B-XH-A_1x04_P2.50mm_Vertical, F.Cu at (132.8, 164.2)
- added JC4: Conn_01x04, Connector_JST:JST_XH_B4B-XH-A_1x04_P2.50mm_Vertical, F.Cu at (149.1, 142.8)
- added JC5: Conn_01x04, Connector_JST:JST_XH_B4B-XH-A_1x04_P2.50mm_Vertical, F.Cu at (134.6, 142.8)
- added JC6: Conn_01x04, Connector_JST:JST_XH_B4B-XH-A_1x04_P2.50mm_Vertical, F.Cu at (120.3, 185.5)
- added JD10: Conn_01x02, Connector_JST:JST_XH_B2B-XH-A_1x02_P2.50mm_Vertical, F.Cu at (168.1, 173.9)
- added JD11: Conn_01x02, Connector_JST:JST_XH_B2B-XH-A_1x02_P2.50mm_Vertical, F.Cu at (203.4, 150.6)
- added JD12: Conn_01x02, Connector_JST:JST_XH_B2B-XH-A_1x02_P2.50mm_Vertical, F.Cu at (177.5, 170.1)
- added JD13: Conn_01x02, Connector_JST:JST_XH_B2B-XH-A_1x02_P2.50mm_Vertical, F.Cu at (194.0, 150.6)
- added JD30: Conn_01x01, Connector_Pin:Pin_D0.9mm_L10.0mm_W2.4mm_FlatFork, F.Cu at (127.0, 170.4)
- added JD31: Conn_01x01, Connector_Pin:Pin_D0.9mm_L10.0mm_W2.4mm_FlatFork, F.Cu at (126.2, 162.8)
- added JD32: Conn_01x01, Connector_Pin:Pin_D0.9mm_L10.0mm_W2.4mm_FlatFork, F.Cu at (169.9, 168.7)
- added JD48: Conn_01x01, Connector_Pin:Pin_D0.9mm_L10.0mm_W2.4mm_FlatFork, F.Cu at (122.5, 170.6)
- added JD49: Conn_01x01, Connector_Pin:Pin_D0.9mm_L10.0mm_W2.4mm_FlatFork, F.Cu at (126.2, 166.6)
- added JD7: Conn_01x02, Connector_JST:JST_XH_B2B-XH-A_1x02_P2.50mm_Vertical, F.Cu at (187.4, 142.8)
- added JD8: Conn_01x02, Connector_JST:JST_XH_B2B-XH-A_1x02_P2.50mm_Vertical, F.Cu at (141.7, 193.5)
- added JD9: Conn_01x02, Connector_JST:JST_XH_B2B-XH-A_1x02_P2.50mm_Vertical, F.Cu at (184.6, 150.6)
- added JP31: Conn_01x02, Connector_JST:JST_XH_B2B-XH-A_1x02_P2.50mm_Vertical, F.Cu at (180.6, 162.3)
- added JP32: Conn_01x02, Connector_JST:JST_XH_B2B-XH-A_1x02_P2.50mm_Vertical, F.Cu at (167.0, 181.8)
- added JP33: Conn_01x02, Connector_JST:JST_XH_B2B-XH-A_1x02_P2.50mm_Vertical, F.Cu at (206.3, 142.8)
- added JP34: Conn_01x02, Connector_JST:JST_XH_B2B-XH-A_1x02_P2.50mm_Vertical, F.Cu at (190.0, 158.3)
- added JP35: Conn_01x02, Connector_JST:JST_XH_B2B-XH-A_1x02_P2.50mm_Vertical, F.Cu at (196.8, 138.5)
- added JP51: Conn_01x02, Connector_JST:JST_XH_B2B-XH-A_1x02_P2.50mm_Vertical, F.Cu at (151.1, 193.5)
- added JP52: Conn_01x02, Connector_JST:JST_XH_B2B-XH-A_1x02_P2.50mm_Vertical, F.Cu at (158.6, 173.9)
- added JP53: Conn_01x02, Connector_JST:JST_XH_B2B-XH-A_1x02_P2.50mm_Vertical, F.Cu at (171.1, 162.3)
- added JP54: Conn_01x02, Connector_JST:JST_XH_B2B-XH-A_1x02_P2.50mm_Vertical, F.Cu at (206.3, 134.9)
- added JP55: Conn_01x02, Connector_JST:JST_XH_B2B-XH-A_1x02_P2.50mm_Vertical, F.Cu at (157.5, 181.8)
- added JX2: Conn_01x03, Connector_JST:JST_XH_B3B-XH-A_1x03_P2.50mm_Vertical, F.Cu at (147.2, 166.2)
- added SQW1: Conn_01x01, Connector_Pin:Pin_D0.9mm_L10.0mm_W2.4mm_FlatFork, F.Cu at (191.2, 137.1)
- added U1: DS1307+, Package_DIP:DIP-8_W7.62mm, F.Cu at (144.8, 180.4)
- added U2: 24LC256, Package_DIP:DIP-8_W7.62mm_LongPads, F.Cu at (171.4, 149.2)
- added U3: W5500, NIC:W5500, F.Cu at (119.1, 160.1)
Connections:
- P1 pad 1: GND -> SDA
- P1 pad 2: GND -> SDA
- P10 pad 1: Net-(P10-Pad1) -> unconnected-(P10-Pad1)
- P11 pad 1: Net-(P11-Pad1) -> unconnected-(P11-Pad1)
- P12 pad 1: Net-(P12-Pad1) -> unconnected-(P12-Pad1)
- P13 pad 1: Net-(P13-Pad1) -> unconnected-(P13-Pad1)
- P2 pad 1: Net-(P2-Pad1) -> unconnected-(P2-Pad1)
- P2 pad 6: GND -> SDA
- P2 pad 7: GND -> SDA
- P5 pad 1: /SCL -> SCL
- P5 pad 2: /SDA -> SDA
- P5 pad 4: GND -> SDA
- P6 pad 7: /1(Tx0) -> unconnected-(P6-Pad7)
- P6 pad 8: /0(Rx0) -> unconnected-(P6-Pad8)
- P8 pad 1: Net-(P8-Pad1) -> unconnected-(P8-Pad1)
- P9 pad 1: Net-(P9-Pad1) -> unconnected-(P9-Pad1)
