File: 001/001.kicad_sch (KiCad schematic)
At the start: 32 parts, among them P1 Digital, P10 CONN_01X01, P11 CONN_01X01, P12 CONN_01X01, P13 CONN_01X01, P2 Power, P3 Analog, P4 Analog, P5 PWM, P6 PWM, P7 Communication, P8 CONN_01X01, P9 CONN_01X01

Commit message: 信号ラベルの見直し中
Parts:
- removed SW?: SW_Push, symbol Switch:SW_Push
- added C3: 100u/35V, symbol Device:C_Polarized_Small
- added D4: D, Diode_THT:D_DO-35_SOD27_P10.16mm_Horizontal, symbol Device:D
- added J1: LCD 2004, Connector_PinHeader_2.54mm:PinHeader_1x16_P2.54mm_Vertical, symbol Connector_Generic:Conn_01x16
- added J2: Relay OUT, Connector_JST:JST_XH_B9B-XH-A_1x09_P2.50mm_Vertical, symbol Connector_Generic:Conn_01x09
- added J5: Conn_01x02, symbol Connector_Generic:Conn_01x02
- added JA0, JA1, JA10, JA11, JA12, JA13, JA14, JA15, JA2, JA3, JA4, JA5, JA6, JA7, JA8, JA9, JX2: Conn_01x03, Connector_JST:JST_XH_B3B-XH-A_1x03_P2.50mm_Vertical, symbol Connector_Generic:Conn_01x03
- added JC1, JC2, JC3, JC4, JC5, JC6: Conn_01x04, Connector_JST:JST_XH_B4B-XH-A_1x04_P2.50mm_Vertical, symbol Connector_Generic:Conn_01x04
- added JD10, JD11, JD12, JD13, JD6, JD7, JD8, JD9, JP31, JP32, JP33, JP34, JP35, JP51, JP52, JP53, JP54, JP55: Conn_01x02, Connector_JST:JST_XH_B2B-XH-A_1x02_P2.50mm_Vertical, symbol Connector_Generic:Conn_01x02
- added JD30, JD31, JD32, JD48, JD49, SQW1: Conn_01x01, Connector_Pin:Pin_D0.9mm_L10.0mm_W2.4mm_FlatFork, symbol Connector_Generic:Conn_01x01
- added RV1: 10k, symbol Device:R_Potentiometer_Small
- added SW1: RESET, symbol Switch:SW_SPST
- added SW2: SW_A, symbol Switch:SW_SPST
- added SW3: SW_B, symbol Switch:SW_SPST
- added SW4: SW_C, symbol Switch:SW_SPST
- added SW5: SW_D, symbol Switch:SW_SPST
- C1, C2: renamed from C?; symbol akizuki:C -> Device:C_Small
- J3: renamed from J?; footprint (none) -> Connector_JST:JST_XH_B7B-XH-A_1x07_P2.50mm_Vertical
- J4: renamed from J?; footprint (none) -> Connector_JST:JST_XH_B5B-XH-A_1x05_P2.50mm_Vertical
- U2: renamed from U?; footprint (none) -> Package_DIP:DIP-8_W7.62mm_LongPads
- U3: renamed from U?; footprint (none) -> NIC:W5500
- gave numbers to parts that had none: 12
Connections:
- net SDA is gone; now on net GND: P5.2 (Pin_2), R2.2, U1.5 (SDA), U2.5 (SDA)
- net +3V3: now also JP31.2 (Pin_2), JP32.2 (Pin_2), JP33.2 (Pin_2), JP34.2 (Pin_2), JP35.2 (Pin_2)
- net +5V: now also C1.1, C3.1, D4.1 (K), J1.15 (Pin_15), J1.2 (Pin_2), J2.9 (Pin_9), JA0.3 (Pin_3), JA1.3 (Pin_3), JA10.3 (Pin_3), JA11.3 (Pin_3), JA12.3 (Pin_3), JA13.3 (Pin_3), JA14.3 (Pin_3), JA15.3 (Pin_3), JA2.3 (Pin_3), JA3.3 (Pin_3), JA4.3 (Pin_3), JA5.3 (Pin_3), JA6.3 (Pin_3), JA7.3 (Pin_3), JA8.3 (Pin_3), JA9.3 (Pin_3), JC1.2 (Pin_2), JC2.2 (Pin_2), JC3.2 (Pin_2), JC4.2 (Pin_2), JC5.2 (Pin_2), JC6.2 (Pin_2), JP51.2 (Pin_2), JP52.2 (Pin_2), JP53.2 (Pin_2), JP54.2 (Pin_2), JP55.2 (Pin_2), RV1.1; no longer C1.2, C2.2
- net 0(Rx0): no longer P6.8 (Pin_8)
- net 1(Tx0): no longer P6.7 (Pin_7)
- net 10(**): now also JD10.2 (Pin_2)
- net 11(**): now also JD11.2 (Pin_2)
- net 12(**): now also JD12.2 (Pin_2)
- net 13(**): now also JD13.2 (Pin_2)
- net 16(Tx2): now also JX2.2 (Pin_2)
- net 17(Rx2): now also JX2.3 (Pin_3)
- net 20(SDA): no longer P7.7 (Pin_7)
- net 21(SCL): no longer P7.8 (Pin_8)
- net 22: now also J2.1 (Pin_1)
- net 23: now also J2.2 (Pin_2)
- net 24: now also J2.3 (Pin_3)
- net 25: now also J2.4 (Pin_4)
- net 26: now also J2.5 (Pin_5)
- net 27: now also J2.6 (Pin_6)
- net 28: now also J2.7 (Pin_7)
- net 29: now also J2.8 (Pin_8)
- net 30: now also JD30.1 (Pin_1)
- net 31: now also JD31.1 (Pin_1)
- net 32: now also JD32.1 (Pin_1)
- net 33: now also SW2.2 (B)
- net 34: now also SW3.2 (B)
- net 35: now also SW4.2 (B)
- net 36: now also SW5.2 (B)
- net 37: no longer P1.20 (Pin_20)
- net 38: now also J1.5 (Pin_5)
- net 39: now also J1.6 (Pin_6)
- net 40: now also J1.7 (Pin_7)
- net 41: now also J1.8 (Pin_8)
- net 42: now also J1.9 (Pin_9)
- net 43: no longer P1.14 (Pin_14)
- net 44: now also J1.11 (Pin_11)
- net 45: no longer P1.12 (Pin_12)
- net 46: now also J1.13 (Pin_13)
- net 47: no longer P1.10 (Pin_10)
- net 48: now also JD48.1 (Pin_1)
- net 49: now also JD49.1 (Pin_1)
- net 6(**): now also JD6.2 (Pin_2)
- net 7(**): now also JD7.2 (Pin_2)
- net 8(**): now also JD8.2 (Pin_2)
- net 9(**): now also JD9.2 (Pin_2)
- net A0: now also JA0.2 (Pin_2)
- net A1: now also JA1.2 (Pin_2)
- net A10: now also JA10.2 (Pin_2)
- net A11: now also JA11.2 (Pin_2)
- net A12: now also JA12.2 (Pin_2)
- net A13: now also JA13.2 (Pin_2)
- net A14: now also JA14.2 (Pin_2)
- net A15: now also JA15.2 (Pin_2)
- net A2: now also JA2.2 (Pin_2)
- net A3: now also JA3.2 (Pin_2)
- net A4: now also JA4.2 (Pin_2)
- net A5: now also JA5.2 (Pin_2)
- net A6: now also JA6.2 (Pin_2)
- net A7: now also JA7.2 (Pin_2)
- net A8: now also JA8.2 (Pin_2)
- net A9: now also JA9.2 (Pin_2)
- net GND: now also C1.2, C3.2, J1.1 (Pin_1), J1.16 (Pin_16), J5.1 (Pin_1), JA0.1 (Pin_1), JA1.1 (Pin_1), JA10.1 (Pin_1), JA11.1 (Pin_1), JA12.1 (Pin_1), JA13.1 (Pin_1), JA14.1 (Pin_1), JA15.1 (Pin_1), JA2.1 (Pin_1), JA3.1 (Pin_1), JA4.1 (Pin_1), JA5.1 (Pin_1), JA6.1 (Pin_1), JA7.1 (Pin_1), JA8.1 (Pin_1), JA9.1 (Pin_1), JC1.1 (Pin_1), JC1.3 (Pin_3), JC2.1 (Pin_1), JC2.3 (Pin_3), JC3.1 (Pin_1), JC3.3 (Pin_3), JC4.1 (Pin_1), JC4.3 (Pin_3), JC5.1 (Pin_1), JC5.3 (Pin_3), JC6.1 (Pin_1), JC6.3 (Pin_3), JD10.1 (Pin_1), JD11.1 (Pin_1), JD12.1 (Pin_1), JD13.1 (Pin_1), JD6.1 (Pin_1), JD7.1 (Pin_1), JD8.1 (Pin_1), JD9.1 (Pin_1), JP31.1 (Pin_1), JP32.1 (Pin_1), JP33.1 (Pin_1), JP34.1 (Pin_1), JP35.1 (Pin_1), JP51.1 (Pin_1), JP52.1 (Pin_1), JP53.1 (Pin_1), JP54.1 (Pin_1), JP55.1 (Pin_1), JX2.1 (Pin_1), RV1.3, SW1.2 (B), SW2.1 (A), SW3.1 (A), SW4.1 (A), SW5.1 (A); no longer C1.1, C2.1
- net IOREF: no longer P2.2 (Pin_2)
- net Reset: now also SW1.1 (A)
- net SCL: now also JC1.4 (Pin_4), JC2.4 (Pin_4), JC3.4 (Pin_4), JC4.4 (Pin_4), JC5.4 (Pin_4), JC6.4 (Pin_4)
- net Vin: no longer P2.8 (Pin_8)
- net at U1.7 (SQW/OUT): now also SQW1.1 (Pin_1)
- new net: D4.2 (A), J5.2 (Pin_2)
- new net DB3: J1.10 (Pin_10), P1.14 (Pin_14)
- new net DB5: J1.12 (Pin_12), P1.12 (Pin_12)
- new net DB7: J1.14 (Pin_14), P1.10 (Pin_10)
- new net RS: J1.4 (Pin_4), P1.20 (Pin_20)
- new net V0: J1.3 (Pin_3), RV1.2
- no-connect marks 12 -> 15
Other:
- note added: "P-00706"
- note added: "P-06063"
- note added: "P-10844"
- moved on the sheet: BT1, D1, D2, D3, R1, R4, R5, R6, U3

Commit message: 回路だいたい出来た。
Parts:
- removed JD6: Conn_01x02, Connector_JST:JST_XH_B2B-XH-A_1x02_P2.50mm_Vertical, symbol Connector_Generic:Conn_01x02
- added SW6: SAFEMODE, symbol Switch:SW_SPST
- BT1: value Battery_Cell -> CR2032
Connections:
- net DB3 is gone; now on net 43: J1.10 (Pin_10), P1.14 (Pin_14)
- net DB5 is gone; now on net 45: J1.12 (Pin_12), P1.12 (Pin_12)
- net DB7 is gone; now on net 47: J1.14 (Pin_14), P1.10 (Pin_10)
- net RS is gone; now on net 37: J1.4 (Pin_4), P1.20 (Pin_20)
- net +5V: now also C2.1
- net 15(Rx3): no longer J3.5 (Pin_5), P7.6 (Pin_6)
- net 20(SDA): now also P7.7 (Pin_7)
- net 21(SCL): now also P7.8 (Pin_8)
- net 3(**): now also SW6.2 (B); no longer D1.1 (K)
- net 6(**): now also D1.1 (K)
- net GND: now also C2.2, SW6.1 (A)
- net IOREF: now also P2.2 (Pin_2)
- net Vin: now also P2.8 (Pin_8)
- net !RESET: no longer names the net of D1.2 (A), J3.1 (Pin_1), R4.2
- net RX: no longer names the net of D2.2 (A), J4.2 (Pin_2), R6.2
- net RX: no longer D3.2 (A), J3.6 (Pin_6), R5.2
- new net: D3.2 (A), J3.6 (Pin_6), R5.2
- new net 19(Rx1): J3.5 (Pin_5), P7.6 (Pin_6)
- no-connect marks 15 -> 10
Other:
- note added: "!RESET"
- note added: "0(Rx0)"
- note added: "1(Tx0)"
- note added: "BL+"
- note added: "BL-"
- note added: "BUSY"
- note added: "DB0"
- note added: "DB1"
- note added: "DB2"
- note added: "DB3"
- note added: "DB4"
- note added: "DB5"
- note added: "DB6"
- note added: "DB7"
- note added: "Ena"
- note added: "GND"
- note added: "R/!W"
- note added: "RS"
- note added: "RX"
- note added: "STATUS"
- note added: "TX"
- note added: "Vdd"
- moved on the sheet: D1, R4
