File: M304.kicad_sch (KiCad schematic)
At the start: 88 parts, among them J1 LCD 2004, J2 Relay OUT, J3 iM920, J4 GPS, J5 POWER IN, P1 Digital, P10 CONN_01X01, P11 CONN_01X01, P12 CONN_01X01, P13 CONN_01X01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

Commit message: Lab Support九州 ヴァージョン
Other:
- company: AMPSD Kyushu Univ. -> Lab Support九州
- title: M304 UECS Controller shield for Arduino MEGA SMANOU2022 -> LY9304 UECS Controller shield for Arduino MEGA
Changed lines of the file:
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@@
 	(paper "A4")
 	(title_block
-		(title "M304 UECS Controller shield for Arduino MEGA SMANOU2022")
-		(date "2022-05-26")
-		(rev "0.01")
-		(company "AMPSD Kyushu Univ.")
-		(comment 1 "RTC I2C")
+		(title "LY9304 UECS Controller shield for Arduino MEGA")
+		(date "2025-01-27")
+		(rev "1.00")
+		(company "Lab Support九州")
 	)
 	(junction
@@
 	(label "21(SCL)"
 		(at 156.21 114.3 0)
-		(fields_autoplaced yes)
 		(effects
 			(font
@@
 	(label "36"
 		(at 151.13 156.21 0)
-		(fields_autoplaced yes)
 		(effects
 			(font
@@
 	(label "17(Rx2)"
 		(at 160.02 104.14 0)
-		(fields_autoplaced yes)
 		(effects
 			(font
@@
 	(label "19(Rx1)"
 		(at 160.02 109.22 0)
-		(fields_autoplaced yes)
 		(effects
 			(font
@@
 	(label "SDA"
 		(at 162.56 41.91 0)
-		(fields_autoplaced yes)
 		(effects
 			(font
@@
 	(label "A14"
 		(at 124.46 111.76 0)
-		(fields_autoplaced yes)
 		(effects
 			(font
@@
 	(label "51(MOSI)"
 		(at 123.19 138.43 0)
-		(fields_autoplaced yes)
 		(effects
 			(font
@@
 	(label "41"
 		(at 132.08 151.13 180)
-		(fields_autoplaced yes)
 		(effects
 			(font
@@
 	(label "43"
 		(at 132.08 148.59 180)
-		(fields_autoplaced yes)
 		(effects
 			(font
@@
 	(label "A3"
 		(at 124.46 80.01 0)
-		(fields_autoplaced yes)
 		(effects
 			(font
@@
 	(label "45"
 		(at 132.08 146.05 180)
-		(fields_autoplaced yes)
 		(effects
 			(font
@@
 	(label "9(**)"
 		(at 160.02 59.69 0)
-		(fields_autoplaced yes)
 		(effects
 			(font
@@
 	(label "GND"
 		(at 254 157.48 0)
-		(fields_autoplaced yes)
 		(effects
 			(font
@@
 	(label "SCL"
 		(at 162.56 39.37 0)
-		(fields_autoplaced yes)
 		(effects
 			(font
@@
 	(label "A8"
 		(at 124.46 96.52 0)
-		(fields_autoplaced yes)
 		(effects
 			(font
@@
 	(label "14(Tx3)"
 		(at 160.02 96.52 0)
-		(fields_autoplaced yes)
 		(effects
 			(font
@@
 	(label "27"
 		(at 125.73 168.91 0)
-		(fields_autoplaced yes)
 		(effects
 			(font
@@
 	(label "12(**)"
 		(at 160.02 52.07 0)
-		(fields_autoplaced yes)
 		(effects
 			(font
@@
 	(label "A5"
 		(at 124.46 85.09 0)
-		(fields_autoplaced yes)
 		(effects
 			(font
@@
 	(label "IOREF"
 		(at 135.89 46.99 180)
-		(fields_autoplaced yes)
 		(effects
 			(font
@@
 	(label "3(**)"
 		(at 160.02 82.55 0)
-		(fields_autoplaced yes)
 		(effects
 			(font
@@
 	(label "Reset"
 		(at 116.84 49.53 0)
-		(fields_autoplaced yes)
 		(effects
 			(font
@@
 	(label "A0"
 		(at 124.46 72.39 0)
-		(fields_autoplaced yes)
 		(effects
 			(font
@@
 	(label "A1"
 		(at 124.46 74.93 0)
-		(fields_autoplaced yes)
 		(effects
 			(font
@@
 	(label "A11"
 		(at 124.46 104.14 0)
-		(fields_autoplaced yes)
 		(effects
 			(font
@@
 	(label "40"
 		(at 151.13 151.13 0)
-		(fields_autoplaced yes)
 		(effects
 			(font
@@
 	(label "53(SS)"
 		(at 123.19 135.89 0)
-		(fields_autoplaced yes)
 		(effects
 			(font
@@
 	(label "30"
 		(at 148.59 163.83 0)
-		(fields_autoplaced yes)
 		(effects
 			(font
@@
 	(label "31"
 		(at 125.73 163.83 0)
-		(fields_autoplaced yes)
 		(effects
 			(font
@@
 	(label "28"
 		(at 151.13 166.37 0)
-		(fields_autoplaced yes)
 		(effects
 			(font
@@
 	(label "44"
 		(at 151.13 146.05 0)
-		(fields_autoplaced yes)
 		(effects
 			(font
@@
 	(label "6(**)"
 		(at 160.02 74.93 0)
-		(fields_autoplaced yes)
 		(effects
 			(font
@@
 	(label "5(**)"
 		(at 160.02 77.47 0)
-		(fields_autoplaced yes)
 		(effects
 			(font
@@
 	(label "37"
 		(at 132.08 156.21 180)
-		(fields_autoplaced yes)
 		(effects
 			(font
@@
 	(label "38"
 		(at 151.13 153.67 0)
-		(fields_autoplaced yes)
 		(effects
 			(font
@@
 	(label "29"
 		(at 125.73 166.37 0)
-		(fields_autoplaced yes)
 		(effects
 			(font
@@
 	(label "18(Tx1)"
 		(at 160.02 106.68 0)
-		(fields_autoplaced yes)
 		(effects
 			(font
@@
 	(label "24"
 		(at 151.13 171.45 0)
-		(fields_autoplaced yes)
 		(effects
 			(font
@@
 	(label "A9"
 		(at 124.46 99.06 0)
-		(fields_autoplaced yes)
 		(effects
 			(font
@@
 	(label "39"
 		(at 132.08 153.67 180)
-		(fields_autoplaced yes)
 		(effects
 			(font
@@
 	(label "22"
 		(at 151.13 173.99 0)
-		(fields_autoplaced yes)
 		(effects
 			(font
@@
 	(label "A15"
 		(at 124.46 114.3 0)
-		(fields_autoplaced yes)
 		(effects
 			(font
@@
 	(label "A6"
 		(at 124.46 87.63 0)
-		(fields_autoplaced yes)
 		(effects
 			(font
@@
 	(label "48"
 		(at 147.32 140.97 0)
-		(fields_autoplaced yes)
 		(effects
 			(font
@@
 	(label "Vin"
 		(at 124.46 43.18 180)
-		(fields_autoplaced yes)
 		(effects
 			(font
@@
 	(label "A7"
 		(at 124.46 90.17 0)
-		(fields_autoplaced yes)
 		(effects
 			(font
@@
 	(label "23"
 		(at 125.73 173.99 0)
-		(fields_autoplaced yes)
 		(effects
 			(font
@@
 	(label "2(**)"
 		(at 160.02 85.09 0)
-		(fields_autoplaced yes)
 		(effects
 			(font
@@
 	(label "49"
 		(at 130.81 140.97 0)
-		(fields_autoplaced yes)
 		(effects
 			(font
@@
 	(label "A13"
 		(at 124.46 109.22 0)
-		(fields_autoplaced yes)
 		(effects
 			(font
@@
 	(label "A2"
 		(at 124.46 77.47 0)
-		(fields_autoplaced yes)
 		(effects
 			(font
@@
 	(label "A12"
 		(at 124.46 106.68 0)
-		(fields_autoplaced yes)
 		(effects
 			(font
@@
 	(label "50(MISO)"
 		(at 151.13 124.46 0)
-		(fields_autoplaced yes)
 		(effects
 			(font
@@
 	(label "52(SCK)"
 		(at 149.86 123.19 180)
-		(fields_autoplaced yes)
 		(effects
 			(font
@@
 	(label "26"
 		(at 151.13 168.91 0)
-		(fields_autoplaced yes)
 		(effects
 			(font
@@
 	(label "47"
 		(at 132.08 143.51 180)
-		(fields_autoplaced yes)
 		(effects
 			(font
@@
 	(label "A4"
 		(at 124.46 82.55 0)
-		(fields_autoplaced yes)
 		(effects
 			(font
@@
 	(label "8(**)"
 		(at 160.02 62.23 0)
-		(fields_autoplaced yes)
 		(effects
 			(font
@@
 	(label "42"
 		(at 151.13 148.59 0)
-		(fields_autoplaced yes)
 		(effects
 			(font
@@
 	(label "A10"
 		(at 124.46 101.6 0)
-		(fields_autoplaced yes)
 		(effects
 			(font
@@
 	(label "7(**)"
 		(at 160.02 72.39 0)
-		(fields_autoplaced yes)
 		(effects
 			(font
@@
 	(label "20(SDA)"
 		(at 156.21 111.76 0)
-		(fields_autoplaced yes)
 		(effects
 			(font
@@
 	(label "16(Tx2)"
 		(at 160.02 101.6 0)
-		(fields_autoplaced yes)
 		(effects
 			(font
@@
 	(label "46"
 		(at 151.13 143.51 0)
-		(fields_autoplaced yes)
 		(effects
 			(font
@@
 	(label "11(**)"
 		(at 160.02 54.61 0)
-		(fields_autoplaced yes)
 		(effects
 			(font
@@
 	(label "4(**)"
 		(at 160.02 80.01 0)
-		(fields_autoplaced yes)
 		(effects
 			(font
@@
 	(label "V0"
 		(at 215.9 129.54 0)
-		(fields_autoplaced yes)
 		(effects
 			(font
@@
 	(label "13(**)"
 		(at 160.02 49.53 0)
-		(fields_autoplaced yes)
 		(effects
 			(font
@@
 	(label "15(Rx3)"
 		(at 160.02 99.06 0)
-		(fields_autoplaced yes)
 		(effects
 			(font
@@
 	(label "10(**)"
 		(at 160.02 57.15 0)
-		(fields_autoplaced yes)
 		(effects
 			(font
@@
 	(label "32"
 		(at 148.59 161.29 0)
-		(fields_autoplaced yes)
 		(effects
 			(font
@@
 	(label "33"
 		(at 129.54 161.29 0)
-		(fields_autoplaced yes)
 		(effects
 			(font
@@
 	(label "34"
 		(at 151.13 158.75 0)
-		(fields_autoplaced yes)
 		(effects
 			(font
@@
 	(label "35"
 		(at 129.54 158.75 0)
-		(fields_autoplaced yes)
 		(effects
 			(font
@@
 	(label "25"
 		(at 125.73 171.45 0)
-		(fields_autoplaced yes)
 		(effects
 			(font
@@
 	(label "AREF"
 		(at 156.21 44.45 0)
-		(fields_autoplaced yes)
 		(effects
 			(font
