File: RTC.kicad_sch (KiCad schematic)
At the start: 5 parts, among them U1 DS1307+, Y1 32.768kHz

Commit message: Lab Support九州 ヴァージョン
Other:
- company: HOLLY&Co.,Ltd. -> Lab Support九州
Changed lines of the file:
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@@
 	(title_block
 		(title "RTC回路")
-		(date "2022-08-02")
+		(date "2025-01-27")
 		(rev "1.00")
-		(company "HOLLY&Co.,Ltd.")
+		(company "Lab Support九州")
 	)
 	(junction
@@
 		(shape bidirectional)
 		(at 172.72 86.36 0)
-		(fields_autoplaced yes)
 		(effects
 			(font
@@
 		(shape input)
 		(at 135.89 57.15 90)
-		(fields_autoplaced yes)
 		(effects
 			(font
@@
 		(shape bidirectional)
 		(at 172.72 96.52 0)
-		(fields_autoplaced yes)
 		(effects
 			(font
@@
 		(shape input)
 		(at 172.72 83.82 0)
-		(fields_autoplaced yes)
-		(effects
-			(font
+		(effects
+			(font
