File: RelayManualSwitch.kicad_sch (KiCad schematic)
At the start: 25 parts, among them SW2-1 SW_SPDT, SW2-2 SW_SPDT, SW2-3 SW_SPDT, SW2-4 SW_SPDT, SW2-5 SW_SPDT, SW2-6 SW_SPDT, SW2-7 SW_SPDT, SW2-8 SW_SPDT, SW2-9 MS611F, U2-1 TLP222G-2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

Commit message: Lab Support九州 ヴァージョン
Other:
- company: (none) -> Lab Support九州
Changed lines of the file:
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@@
 	(title_block
 		(title "Relay Control AUTO/MANUAL")
-		(date "2022-07-08")
+		(date "2025-01-27")
 		(rev "1.00")
+		(company "Lab Support九州")
 	)
 	(junction
@@
 		(shape input)
 		(at 193.04 148.59 0)
-		(fields_autoplaced yes)
 		(effects
 			(font
@@
 		(shape input)
 		(at 193.04 111.76 0)
-		(fields_autoplaced yes)
 		(effects
 			(font
@@
 		(shape input)
 		(at 193.04 151.13 0)
-		(fields_autoplaced yes)
 		(effects
 			(font
@@
 		(shape output)
 		(at 50.8 96.52 180)
-		(fields_autoplaced yes)
 		(effects
 			(font
@@
 		(shape output)
 		(at 50.8 106.68 180)
-		(fields_autoplaced yes)
 		(effects
 			(font
@@
 		(shape input)
 		(at 193.04 96.52 0)
-		(fields_autoplaced yes)
 		(effects
 			(font
@@
 		(shape input)
 		(at 248.285 52.705 0)
-		(fields_autoplaced yes)
 		(effects
 			(font
@@
 		(shape output)
 		(at 50.8 111.76 180)
-		(fields_autoplaced yes)
 		(effects
 			(font
@@
 		(shape input)
 		(at 248.92 30.48 0)
-		(fields_autoplaced yes)
 		(effects
 			(font
@@
 		(shape input)
 		(at 193.04 101.6 0)
-		(fields_autoplaced yes)
 		(effects
 			(font
@@
 		(shape output)
 		(at 50.8 170.18 180)
-		(fields_autoplaced yes)
 		(effects
 			(font
@@
 		(shape input)
 		(at 193.04 106.68 0)
-		(fields_autoplaced yes)
 		(effects
 			(font
@@
 		(shape output)
 		(at 50.8 165.1 180)
-		(fields_autoplaced yes)
 		(effects
 			(font
@@
 		(shape input)
 		(at 248.158 66.04 0)
-		(fields_autoplaced yes)
 		(effects
 			(font
@@
 		(shape output)
 		(at 50.8 101.6 180)
-		(fields_autoplaced yes)
 		(effects
 			(font
@@
 		(shape input)
 		(at 193.04 146.05 0)
-		(fields_autoplaced yes)
 		(effects
 			(font
@@
 		(shape output)
 		(at 50.8 160.02 180)
-		(fields_autoplaced yes)
 		(effects
 			(font
@@
 		(shape input)
 		(at 193.04 153.67 0)
-		(fields_autoplaced yes)
 		(effects
 			(font
@@
 		(shape output)
 		(at 50.8 175.26 180)
-		(fields_autoplaced yes)
-		(effects
-			(font
+		(effects
+			(font
